File: Chillboard.kicad_pcb (KiCad board)
At the start: 2 copper layers, 335.6 x 202.9 mm, 199 parts, among them SW1 SW_Push, SW10 SW_Push, SW11 SW_Push, SW12 SW_Push, SW13 SW_Push, SW14 SW_Push, SW15 SW_Push, SW16 SW_Push, SW17 SW_Push, SW18 SW_Push, SW19 SW_Push, SW2 SW_Push, SW20 SW_Push, SW21 SW_Push, SW22 SW_Push, SW23 SW_Push, SW24 SW_Push, SW25 SW_Push, SW26 SW_Push, SW27 SW_Push, SW28 SW_Push, SW29 SW_Push, SW3 SW_Push, SW30 SW_Push, SW31 SW_Push, SW32 SW_Push, SW33 SW_Push, SW34 SW_Push, SW35 SW_Push, SW36 SW_Push, SW37 SW_Push, SW38 SW_Push, SW39 SW_Push, SW4 SW_Push, SW40 SW_Push, SW41 SW_Push, SW42 SW_Push, SW43 RotaryEncoder, SW44 RotaryEncoder, SW5 SW_Push, SW6 SW_Push, SW7 SW_Push, SW8 SW_Push, SW9 SW_Push, U1 XIAO-nRF52840-SMD, U2 XIAO-nRF52840-SMD, U3 PCF8574AP, U4 PCF8574AP

Commit message: done
Parts:
- BO1, BO2, BO3: footprint MountingHole:mouse-bite-5mm-slot -> mousebite:mouse-bite-5mm-slot
- C1, C10, C2, C9, H1, H3, H9, R1, R3, R5, TP3, TP4: moved to B.Cu
- D1, D10, D11, D12, D13, D14, D15, D16, D17, D18, D19, D2, D20, D21, D22, D23, D24, D25, D26, D27, D28, D29, D3, D30, D31, D32, D33, D34, D35, D36, D37, D38, D39, D4, D40, D41, D42, D5, D6, D7, D8, D9: footprint Diode_THT:D_DO-35_SOD27_P7.62mm_Horizontal -> Diode_SMD:D_SOD-123; moved to B.Cu
- D43, D44, D45, D46, D47, D48, D49, D50, D51, D52, D53, D54, D55, D56, D57, D58, D59, D60, D61, D62, D63, D64, D65, D66, D67, D68, D69, D70, D71, D72, D73, D74, D75, D76, D77, D78, D79, D80, D81, D82, D83, D84: footprint LED_SMD:MX_SK6812MINI-E_REV -> PCM_marbastlib-various:LED_6028R; moved to B.Cu
- OLED1, OLED2: footprint Display:SSD1306-0.91-OLED-4pin-128x32 -> KiCad-SSD1306-0.91-OLED-4pin-128x32.pretty-master:SSD1306-0.91-OLED-4pin-128x32
- PIR1, PIR2: footprint Sensor_Motion:BS412 -> BS412:BS412
- SW1, SW10, SW11, SW12, SW13, SW14, SW15, SW16, SW17, SW18, SW19, SW2, SW20, SW21, SW22, SW23, SW24, SW25, SW26, SW27, SW28, SW29, SW3, SW30, SW31, SW32, SW33, SW34, SW35, SW36, SW37, SW38, SW39, SW4, SW40, SW41, SW42, SW5, SW6, SW9: footprint PCM_marbastlib-mx:SW_MX_1u -> marbastlib-choc:SW_choc_v1_HS_CPG135001S30_1u; moved to B.Cu
- SW7, SW8: footprint PCM_marbastlib-mx:SW_MX_1u -> marbastlib-choc:SW_choc_v1_HS_CPG135001S30_1.5u; moved to B.Cu
- TP1, TP2: value TestPoint -> VBAT; moved to B.Cu
- U1, U2: footprint RF_WiFi:modified-XIAO-nRF52840-SMD -> modified-xiao:modified-XIAO-nRF52840-SMD
- moved D83 258.3 mm to (484.2, 117.0)
- moved SW41 237.0 mm to (465.3, 102.6), turned to 180 degrees
- moved H1 233.4 mm to (474.8, 112.2), turned to 180 degrees
- moved D41 232.0 mm to (468.8, 112.3)
- moved C38 227.2 mm to (451.7, 111.4), turned to 180 degrees
- moved C2 225.5 mm to (52.5, 58.0), turned to 180 degrees
- moved C41 225.1 mm to (489.7, 116.2), turned to 180 degrees
- moved D64 220.7 mm to (484.2, 97.9)
- moved D63 219.7 mm to (465.2, 97.9)
- moved D34 212.1 mm to (489.1, 110.9), turned to 0 degrees
- moved C40 208.7 mm to (470.7, 97.0), turned to 180 degrees
- moved C17 208.0 mm to (432.7, 90.0), turned to 180 degrees
- moved D3 197.5 mm to (422.5, 144.7), turned to 0 degrees
- moved SW3 197.3 mm to (417.8, 136.4), turned to 180 degrees
- moved D25 195.6 mm to (470.1, 129.8), turned to 180 degrees
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Connections:
- D41 pad 1: /left/ROW5 -> ROW5
- D42 pad 1: /right/ROW5 -> ROW5
- D43 pad 1: Net-(D43-DOUT) -> +5V
- D43 pad 2: GND -> Net-(D43-DOUT)
- D43 pad 4: +5V -> GND
- D44 pad 1: Net-(D44-DOUT) -> +5V
- D44 pad 2: GND -> Net-(D44-DOUT)
- D44 pad 4: +5V -> GND
- D45 pad 1: Net-(D45-DOUT) -> +5V
- D45 pad 2: GND -> Net-(D45-DOUT)
- D45 pad 4: +5V -> GND
- D46 pad 1: Net-(D46-DOUT) -> +5V
- D46 pad 2: GND -> Net-(D46-DOUT)
- D46 pad 4: +5V -> GND
- D47 pad 1: Net-(D47-DOUT) -> +5V
- D47 pad 2: GND -> Net-(D47-DOUT)
- D47 pad 4: +5V -> GND
- D48 pad 1: Net-(D48-DOUT) -> +5V
- D48 pad 2: GND -> Net-(D48-DOUT)
- D48 pad 4: +5V -> GND
- D49 pad 1: Net-(D49-DOUT) -> +5V
- D49 pad 2: GND -> Net-(D49-DOUT)
- D49 pad 4: +5V -> GND
- D50 pad 1: Net-(D50-DOUT) -> +5V
- D50 pad 2: GND -> Net-(D50-DOUT)
- D50 pad 4: +5V -> GND
- D51 pad 1: Net-(D51-DOUT) -> +5V
- D51 pad 2: GND -> Net-(D51-DOUT)
- D51 pad 4: +5V -> GND
- D52 pad 1: Net-(D52-DOUT) -> +5V
- D52 pad 2: GND -> Net-(D52-DOUT)
- D52 pad 4: +5V -> GND
- D53 pad 1: Net-(D53-DOUT) -> +5V
- D53 pad 2: GND -> Net-(D53-DOUT)
- D53 pad 4: +5V -> GND
- D54 pad 1: Net-(D54-DOUT) -> +5V
- D54 pad 2: GND -> Net-(D54-DOUT)
- D54 pad 4: +5V -> GND
- D55 pad 1: Net-(D55-DOUT) -> +5V
- D55 pad 2: GND -> Net-(D55-DOUT)
- D55 pad 4: +5V -> GND
- D56 pad 1: Net-(D56-DOUT) -> +5V
- D56 pad 2: GND -> Net-(D56-DOUT)
- D56 pad 4: +5V -> GND
- D57 pad 1: Net-(D57-DOUT) -> +5V
- D57 pad 2: GND -> Net-(D57-DOUT)
- D57 pad 4: +5V -> GND
- D58 pad 1: Net-(D58-DOUT) -> +5V
- D58 pad 2: GND -> Net-(D58-DOUT)
- D58 pad 4: +5V -> GND
- D59 pad 1: Net-(D59-DOUT) -> +5V
- D59 pad 2: GND -> Net-(D59-DOUT)
- D59 pad 4: +5V -> GND
- D60 pad 1: Net-(D60-DOUT) -> +5V
- D60 pad 2: GND -> Net-(D60-DOUT)
- D60 pad 4: +5V -> GND
- D61 pad 1: Net-(D61-DOUT) -> +5V
- D61 pad 2: GND -> Net-(D61-DOUT)
- D61 pad 4: +5V -> GND
- D62 pad 1: Net-(D62-DOUT) -> +5V
- D62 pad 2: GND -> Net-(D62-DOUT)
- D62 pad 4: +5V -> GND
- D63 pad 1: Net-(D63-DOUT) -> +5V
- D63 pad 2: GND -> Net-(D63-DOUT)
- D63 pad 4: +5V -> GND
- D64 pad 1: Net-(D64-DOUT) -> +5V
- D64 pad 2: GND -> Net-(D64-DOUT)
- D64 pad 4: +5V -> GND
- D65 pad 1: Net-(D65-DOUT) -> +5V
- D65 pad 2: GND -> Net-(D65-DOUT)
- D65 pad 4: +5V -> GND
- D66 pad 1: Net-(D66-DOUT) -> +5V
- D66 pad 2: GND -> Net-(D66-DOUT)
- D66 pad 4: +5V -> GND
- D67 pad 1: Net-(D67-DOUT) -> +5V
- D67 pad 2: GND -> Net-(D67-DOUT)
- D67 pad 4: +5V -> GND
- D68 pad 1: Net-(D68-DOUT) -> +5V
- D68 pad 2: GND -> Net-(D68-DOUT)
- D68 pad 4: +5V -> GND
- D69 pad 1: Net-(D69-DOUT) -> +5V
- D69 pad 2: GND -> Net-(D69-DOUT)
- D69 pad 4: +5V -> GND
- D70 pad 1: Net-(D70-DOUT) -> +5V
- D70 pad 2: GND -> Net-(D70-DOUT)
- D70 pad 4: +5V -> GND
- D71 pad 1: Net-(D71-DOUT) -> +5V
- D71 pad 2: GND -> Net-(D71-DOUT)
- D71 pad 4: +5V -> GND
- D72 pad 1: Net-(D72-DOUT) -> +5V
- D72 pad 2: GND -> Net-(D72-DOUT)
- D72 pad 4: +5V -> GND
- D73 pad 1: Net-(D73-DOUT) -> +5V
- D73 pad 2: GND -> Net-(D73-DOUT)
- D73 pad 4: +5V -> GND
- D74 pad 1: Net-(D74-DOUT) -> +5V
- D74 pad 2: GND -> Net-(D74-DOUT)
- D74 pad 4: +5V -> GND
- D75 pad 1: Net-(D75-DOUT) -> +5V
- D75 pad 2: GND -> Net-(D75-DOUT)
- D75 pad 4: +5V -> GND
- D76 pad 1: Net-(D76-DOUT) -> +5V
- D76 pad 2: GND -> Net-(D76-DOUT)
- D76 pad 4: +5V -> GND
- D77 pad 1: Net-(D77-DOUT) -> +5V
- D77 pad 2: GND -> Net-(D77-DOUT)
- D77 pad 4: +5V -> GND
- D78 pad 1: Net-(D78-DOUT) -> +5V
- D78 pad 2: GND -> Net-(D78-DOUT)
- D78 pad 4: +5V -> GND
- D79 pad 1: Net-(D79-DOUT) -> +5V
- D79 pad 2: GND -> Net-(D79-DOUT)
- D79 pad 4: +5V -> GND
- D80 pad 1: Net-(D80-DOUT) -> +5V
- D80 pad 2: GND -> Net-(D80-DOUT)
- D80 pad 4: +5V -> GND
- D81 pad 1: Net-(D81-DOUT) -> +5V
- D81 pad 2: GND -> Net-(D81-DOUT)
- D81 pad 4: +5V -> GND
- D82 pad 1: Net-(D82-DOUT) -> +5V
- D82 pad 2: GND -> Net-(D82-DOUT)
- D82 pad 4: +5V -> GND
- D83 pad 1: unconnected-(D83-DOUT-Pad1) -> +5V
- D83 pad 2: GND -> unconnected-(D83-DOUT-Pad2)
- D83 pad 4: +5V -> GND
- D84 pad 1: unconnected-(D84-DOUT-Pad1) -> +5V
- D84 pad 2: GND -> unconnected-(D84-DOUT-Pad2)
- D84 pad 4: +5V -> GND
- OLED1 pad 3: Net-(OLED1-SDA) -> OLED_SDA
- OLED1 pad 4: Net-(OLED1-SCL) -> OLED_SCL
- OLED2 pad 3: Net-(OLED2-SDA) -> OLED_SDA
- OLED2 pad 4: Net-(OLED2-SCL) -> OLED_SCL
- PIR1 pad 3: +3.3V -> +3V3
- PIR1 pad 4: Net-(PIR1-OUT) -> PIR_OUT
- PIR2 pad 3: +3.3V -> +3V3
- PIR2 pad 4: Net-(PIR2-OUT) -> PIR_OUT
- R1 pad 1: /left/BACKLIGHT_LED -> BACKLIGHT_LED
- R2 pad 1: /right/BACKLIGHT_LED -> BACKLIGHT_LED
- R3 pad 1: /left/VBAT -> VBAT
- R3 pad 2: /left/BAT_PIN -> BAT_PIN
- R4 pad 1: /right/VBAT -> VBAT
- R4 pad 2: /right/BAT_PIN -> BAT_PIN
- R5 pad 2: /left/BAT_PIN -> BAT_PIN
- R6 pad 2: /right/BAT_PIN -> BAT_PIN
- SW1 pad 1: /left/COL1 -> COL1
- SW10 pad 1: /left/COL2 -> COL2
- SW11 pad 1: /left/COL2 -> COL2
- SW12 pad 1: /left/COL2 -> COL2
- SW13 pad 1: /right/COL2 -> COL2
- SW14 pad 1: /right/COL2 -> COL2
- SW15 pad 1: /right/COL2 -> COL2
- SW16 pad 1: /right/COL2 -> COL2
- SW17 pad 1: /left/COL3 -> COL3
- SW18 pad 1: /left/COL3 -> COL3
- SW19 pad 1: /left/COL3 -> COL3
- SW2 pad 1: /right/COL1 -> COL1
- SW20 pad 1: /left/COL3 -> COL3
- SW21 pad 1: /right/COL3 -> COL3
- SW22 pad 1: /right/COL3 -> COL3
- SW23 pad 1: /right/COL3 -> COL3
- SW24 pad 1: /right/COL3 -> COL3
- SW25 pad 1: /left/COL4 -> COL4
- SW26 pad 1: /left/COL4 -> COL4
- SW27 pad 1: /left/COL4 -> COL4
- SW28 pad 1: /left/COL4 -> COL4
- SW29 pad 1: /right/COL4 -> COL4
- SW3 pad 1: /left/COL1 -> COL1
- SW30 pad 1: /right/COL4 -> COL4
- SW31 pad 1: /right/COL4 -> COL4
- SW32 pad 1: /right/COL4 -> COL4
- SW33 pad 1: /left/COL5 -> COL5
- SW34 pad 1: /left/COL5 -> COL5
- SW35 pad 1: /left/COL5 -> COL5
- SW36 pad 1: /left/COL5 -> COL5
- SW37 pad 1: /right/COL5 -> COL5
- SW38 pad 1: /right/COL5 -> COL5
- SW39 pad 1: /right/COL5 -> COL5
- SW4 pad 1: /right/COL1 -> COL1
- SW40 pad 1: /right/COL5 -> COL5
- SW41 pad 1: /left/COL5 -> COL5
- SW42 pad 1: /right/COL5 -> COL5
- SW43 pad A: /left/ROT_A -> ROT_A
- SW43 pad B: /left/ROT_B -> ROT_B
- SW44 pad A: /right/ROT_A -> ROT_A
- SW44 pad B: /right/ROT_B -> ROT_B
- SW5 pad 1: /left/COL1 -> COL1
- SW6 pad 1: /right/COL1 -> COL1
- SW7 pad 1: /left/COL1 -> COL1
- SW8 pad 1: /right/COL1 -> COL1
- SW9 pad 1: /left/COL2 -> COL2
- TP1 pad 1: /left/VBAT -> VBAT
- TP2 pad 1: /right/VBAT -> VBAT
- U1 pad 1: /left/BAT_PIN -> BAT_PIN
- U1 pad 12: unconnected-(U1-3V3-Pad12) -> +3V3
- U1 pad 14: unconnected-(U1-5V-Pad14) -> +5V
- U1 pad 15: /left/VBAT -> VBAT
- U1 pad 2: /left/COL1 -> COL1
- U1 pad 3: /left/COL2 -> COL2
- U1 pad 4: /left/COL3 -> COL3
- U1 pad 5: /left/EXP_SDA -> EXP_SDA
- U1 pad 6: /left/EXP_SCL -> EXP_SCL
- U1 pad 7: /left/ROW5 -> ROW5
- U2 pad 1: /right/BAT_PIN -> BAT_PIN
- U2 pad 12: unconnected-(U2-3V3-Pad12) -> +3V3
- U2 pad 14: unconnected-(U2-5V-Pad14) -> +5V
- U2 pad 15: /right/VBAT -> VBAT
- U2 pad 2: /right/COL1 -> COL1
- U2 pad 3: /right/COL2 -> COL2
- U2 pad 4: /right/COL3 -> COL3
- U2 pad 5: /right/EXP_SDA -> EXP_SDA
- U2 pad 6: /right/EXP_SCL -> EXP_SCL
- U2 pad 7: /right/ROW5 -> ROW5
- U3 pad 10: /left/ROT_B -> ROT_B
- U3 pad 11: Net-(OLED1-SDA) -> OLED_SDA
- U3 pad 12: Net-(OLED1-SCL) -> OLED_SCL
- U3 pad 14: /left/EXP_SCL -> EXP_SCL
- U3 pad 15: /left/EXP_SDA -> EXP_SDA
- U3 pad 4: /left/COL4 -> COL4
- U3 pad 5: /left/COL5 -> COL5
- U3 pad 6: /left/BACKLIGHT_LED -> BACKLIGHT_LED
- U3 pad 7: Net-(PIR1-OUT) -> PIR_OUT
- U3 pad 9: /left/ROT_A -> ROT_A
- U4 pad 10: /right/ROT_B -> ROT_B
- U4 pad 11: Net-(OLED2-SDA) -> OLED_SDA
- U4 pad 12: Net-(OLED2-SCL) -> OLED_SCL
- U4 pad 14: /right/EXP_SCL -> EXP_SCL
- U4 pad 15: /right/EXP_SDA -> EXP_SDA
- U4 pad 4: /right/COL4 -> COL4
- U4 pad 5: /right/COL5 -> COL5
- U4 pad 6: /right/BACKLIGHT_LED -> BACKLIGHT_LED
- U4 pad 7: Net-(PIR2-OUT) -> PIR_OUT
- U4 pad 9: /right/ROT_A -> ROT_A
Routing:
- net GND: track 100.8 -> 1762.9 mm, vias 12 -> 63
- net +5V: track 1013.2 -> 1410.4 mm, vias 4 -> 3
- net COL4: track 0.00 -> 382.3 mm, vias 0 -> 4
- net COL1: track 0.00 -> 352.8 mm, vias 0 -> 4
- net ROW5: track 0.00 -> 324.1 mm, vias 0 -> 3
- net COL5: track 0.00 -> 310.3 mm
- net COL3: track 0.00 -> 257.0 mm, vias 0 -> 4
- net BAT_PIN: track 0.00 -> 237.1 mm, vias 0 -> 2
- net COL2: track 0.00 -> 212.1 mm, vias 0 -> 2
- net /right/COL5: track 201.1 -> 0.00 mm
- net /left/EXP_SCL: track 196.2 -> 0.00 mm
- net /right/EXP_SCL: track 196.2 -> 0.00 mm
- net /right/ROT_B: track 180.8 -> 0.00 mm
- net /left/ROT_B: track 180.8 -> 0.00 mm
- net /right/ROT_A: track 179.2 -> 0.00 mm, vias 4 -> 0
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- removed copper zone on B.Cu, net GND
Other:
- board size 335.6 x 202.9 mm -> 480.9 x 112 mm

Commit message: fdhshfadshkfdsahhfadshjkfds
Parts:
- added H2: MountingHole, MountingHole:MountingHole_2.1mm, F.Cu at (118.9, 110.6)
- BO1, BO2, BO3: footprint mousebite:mouse-bite-5mm-slot -> Panelization.pretty-master:mouse-bite-3mm-slot
- H1, H3, H9: moved to F.Cu
- R1: footprint Resistor_THT:R_Axial_DIN0207_L6.3mm_D2.5mm_P10.16mm_Horizontal -> Resistor_THT:R_Axial_DIN0207_L6.3mm_D2.5mm_P7.62mm_Horizontal; moved to F.Cu
- R2: footprint Resistor_THT:R_Axial_DIN0207_L6.3mm_D2.5mm_P10.16mm_Horizontal -> Resistor_THT:R_Axial_DIN0207_L6.3mm_D2.5mm_P7.62mm_Horizontal; moved to B.Cu
- R3, R4, R5, R6: footprint Resistor_THT:R_Axial_DIN0207_L6.3mm_D2.5mm_P10.16mm_Horizontal -> Resistor_SMD:R_0805_2012Metric
- moved R5 188.6 mm to (172.2, 111.9)
- moved C15 188.5 mm to (250.0, 92.6)
- moved C16 188.5 mm to (213.3, 113.8)
- moved C25 188.5 mm to (206.8, 76.0)
- moved C39 188.5 mm to (207.3, 95.2)
- moved C5 188.5 mm to (187.8, 131.0)
- moved C9 188.5 mm to (226.3, 73.7)
- moved D10 188.5 mm to (224.4, 107.5)
- moved D17 188.5 mm to (247.4, 64.3)
- moved D20 188.5 mm to (224.3, 69.5)
- moved D45 188.5 mm to (239.6, 53.0)
- moved D54 188.5 mm to (201.3, 76.7)
- moved D66 188.5 mm to (208.1, 116.0)
- moved H3 188.5 mm to (230.3, 69.5), turned to 0 degrees
- moved PIR1 188.5 mm to (165.3, 80.5)
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Routing:
- net Net-(D51-DOUT): track 0.00 -> 107.1 mm, vias 0 -> 2
- net +5V: track 1410.4 -> 1390.6 mm
- net BAT_PIN: track 237.1 -> 218.2 mm, vias 2 -> 3
- net ROW5: track 324.1 -> 305.9 mm, vias 3 -> 2
- net Net-(D43-DIN): track 113.2 -> 130.5 mm
- net Net-(D28-A): track 21.1 -> 5.48 mm
- net GND: track 1762.9 -> 1748.7 mm, vias 63 -> 61
- net BACKLIGHT_LED: track 82.9 -> 72.9 mm
- net Net-(D67-DOUT): track 50.7 -> 42.0 mm
- net VBAT: track 150.0 -> 155.5 mm, vias 2 -> 1
- net /right/ROW1: track 239.5 -> 234.4 mm, vias 4 -> 5
- net Net-(D1-A): track 19.3 -> 14.3 mm
- net Net-(D20-A): track 0.00 -> 1.98 mm
- net Net-(D44-DIN): track 87.4 -> 85.8 mm
Other:
- board size 480.9 x 112 mm -> 303.7 x 94 mm
